File: tutorial3088.kicad_sch (KiCad schematic)
At the start: 33 parts

Commit message: Add files via upload
Parts:
- removed R?: R_Small, symbol Device:R_Small
- added C?: 330nF, symbol Device:C
- added D? (x4): D, symbol Device:D
- added Q? (x12): Q_NPN_BCE, symbol Device:Q_NPN_BCE
- added Q? (x4): Q_PNP_BCE, symbol Device:Q_PNP_BCE
- added R?: 120k, symbol Device:R
- added R?: 4.7M, symbol Device:R
- added R? (x2): 15, symbol Device:R_Small
- added R? (x5): 120, symbol Device:R_Small
- added R? (x2): 100, symbol Device:R_Small
- added R?: 27, symbol Device:R
- added R? (x4): 2.6k, symbol Device:R_Small
- added R?: R, symbol Device:R
- added R?: 12, symbol Device:R
- added R?: 1M, symbol Device:R
- added R?: 2.2M, symbol Device:R
- added U?: INA219AxD, Package_SO:SOIC-8_3.9x4.9mm_P1.27mm, symbol Analog_ADC:INA219AxD
- added U?: LM7806_TO220, Package_TO_SOT_THT:TO-220-3_Vertical, symbol Regulator_Linear:LM7806_TO220
- C? (x2): value C -> 4.7uF
- R? (x2): value R_Small -> 2.6k
- R? (x2): value R_Small -> 15
- R?: value R -> 1.5M
- R?: value R -> 2k
- R?: value R_Small -> 120
- R?: value R -> 120k
- R?: value R -> 10k
Connections:
- net 3v3: now also D?.1 (K), D?.1 (K)
- net Earth: now also C?.2, D?.2 (A), D?.2 (A), Q?.3 (E), Q?.3 (E), Q?.3 (E), Q?.3 (E), Q?.3 (E), Q?.3 (E), Q?.3 (E), Q?.3 (E), R?.2, R?.2, U?.2 (GND)
- net motor control: now also Q?.1 (B), Q?.1 (B), R?.1, R?.1
- net motor control 2: now also Q?.1 (B), Q?.1 (B), R?.1, R?.1
- net at M?.1 (+), Q?.2 (C), Q?.2 (C): now also D?.1 (K), D?.2 (A)
- net at M?.2 (-), Q?.2 (C), Q?.2 (C): now also D?.1 (K), D?.2 (A)
- net Vin-3.2v: now reaches C?.1, L?.1, Q?.1 (D), R?.1, U?.5 (VIN), U?.6 (EN), U?.8 (PS)
- net motor2_B_out: now reaches J?.1 (Pin_1)
- net motor4_CTRL2: now reaches J?.10 (Pin_10)
- net EXT_LOAD2_OUT: now reaches J?.11 (Pin_11)
- net USART2_TX: now reaches J?.12 (Pin_12)
- net FAST_CHARGE_CTRL: now reaches J?.13 (Pin_13)
- net Battery: now reaches J?.14 (Pin_14)
- net .: now reaches J?.15 (Pin_15)
- net I2C1_SCL: now reaches J?.16 (Pin_16)
- net I2C1_SDA: now reaches J?.17 (Pin_17)
- net 3V3 out: now reaches J?.18 (Pin_18)
- net GND: now reaches J?.19 (Pin_19)
- net GND: now also J?.23 (Pin_23)
- net motor2_A_out: now reaches J?.2 (Pin_2)
- net 5V out: now reaches J?.20 (Pin_20)
- net EXT_LOAD1_OUT: now reaches J?.21 (Pin_21)
- net HV: now reaches J?.22 (Pin_22)
- net motor3_CTRL1: now reaches J?.24 (Pin_24)
- net CTRL_EXT_LOAD1: now reaches J?.25 (Pin_25)
- net motor3_CTRL2: now reaches J?.26 (Pin_26)
- net motor3_A_OUT: now reaches J?.27 (Pin_27)
- net motor1_CTRL1: now reaches J?.28 (Pin_28)
- net motor3_B_OUT: now reaches J?.29 (Pin_29)
- net motor4_A_out: now reaches J?.3 (Pin_3)
- net motor1_CTRL2: now reaches J?.30 (Pin_30)
- net motor1_B_OUT: now reaches J?.31 (Pin_31)
- net motor1_A_OUT: now reaches J?.32 (Pin_32)
- net motor2_CTRL1: now reaches J?.4 (Pin_4)
- net motor4_B_out: now reaches J?.5 (Pin_5)
- net motor2_CTRL2: now reaches J?.6 (Pin_6)
- net CTRL_EXT_LOAD2: now reaches J?.7 (Pin_7)
- net motor4_CTRL1: now reaches J?.8 (Pin_8)
- net USART2_RX: now reaches J?.9 (Pin_9)
- net at Q?.3 (E): now also R?.1
- net at D?.2 (A), J?.A4 (VBUS), J?.A9 (VBUS)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: now also C?.1, U?.1 (VI); no longer C?.1, U?.4 (VDD)
- net at J?.A5 (CC1): no longer J?.B5 (CC2)
- net at J?.A6 (D+), J?.B6 (D+): no longer J?.A7 (D-), J?.B7 (D-)
- net at J?.A8 (SBU1): no longer J?.B8 (SBU2)
- net at Q?.1 (B): now also R?.2
- net Vout: no longer names the net of U?.10 (FB)
- net Vout: now also R?.1, R?.2; no longer U?.2 (VOUT)
- new net: Q?.1 (B), R?.2 (x12)
- new net: U?.2 (A0), U?.6 (GND)
- new net: Q?.2 (C), R?.1 (x4)
- new net: C?.1, U?.3 (VO), U?.4 (VDD)
- new net: Q?.3 (E), R?.1 (x4)
- new net: R?.1, R?.2
- new net: J?.A7 (D-), J?.B7 (D-)
- new net 3v3 out: U?.1 (A1)
- new net 3v3in: R?.1, U?.8 (IN+)
- new net INA219 out: R?.2, U?.7 (IN-)
- new net Vout_3.3v: R?.1, R?.2
- new net Vout_5v: R?.1, R?.1, U?.2 (VOUT)
- new net Vss: Q?.2 (C), Q?.2 (C), Q?.2 (C), Q?.2 (C), Q?.3 (E), Q?.3 (E), Q?.3 (E), Q?.3 (E)
- new net motor_in: Q?.2 (C), Q?.2 (C), Q?.2 (C), Q?.2 (C)
- new net motor_out: Q?.2 (C), Q?.2 (C), Q?.2 (C), Q?.2 (C)
- new net pin3: U?.4 (SCL)
- new net pin4: U?.3 (SDA)
- no-connect marks 1 -> 5
Other:
- note added: "200mA output"
- note added: "500mA out"
- note added: "when battery output is 3.2, vout drops to zero"
- moved on the sheet: J?

Commit message: Add files via upload
Parts:
- removed C?: 22uF, symbol Device:C
- removed C?: 1uF, symbol Device:C
- removed C? (x3): 4.7uF, symbol Device:C
- removed C?: 330nF, symbol Device:C
- removed D? (x4): D, symbol Device:D
- removed D?: D_Schottky, symbol Device:D_Schottky
- removed J?: USB_C_Receptacle_USB2.0, symbol Connector:USB_C_Receptacle_USB2.0
- removed L?: 2.2uH, symbol Device:L
- removed M?: Motor_DC, symbol Motor:Motor_DC
- removed Q? (x18): Q_NPN_BCE, symbol Device:Q_NPN_BCE
- removed Q? (x6): Q_PNP_BCE, symbol Device:Q_PNP_BCE
- removed Q?: Q_PMOS_DSG, symbol Device:Q_PMOS_DSG
- removed R? (x2): 120k, symbol Device:R
- removed R?: 4.7M, symbol Device:R
- removed R? (x6): 2.6k, symbol Device:R_Small
- removed R? (x4): 15, symbol Device:R_Small
- removed R? (x6): 120, symbol Device:R_Small
- removed R? (x2): 100, symbol Device:R_Small
- removed R?: 27, symbol Device:R
- removed R?: R, symbol Device:R
- removed R?: 1.5M, symbol Device:R
- removed R?: 2k, symbol Device:R
- removed R?: 12, symbol Device:R
- removed R?: 1M, symbol Device:R
- removed R?: 2.2M, symbol Device:R
- removed R?: 10k, symbol Device:R
- removed TP? (x2): TestPoint, symbol Connector:TestPoint
- removed U?: TPS61200DRC, Package_SON:Texas_S-PVSON-N10_ThermalVias, symbol Regulator_Switching:TPS61200DRC
- removed U?: MCP73831-2-OT, Package_TO_SOT_SMD:SOT-23-5, symbol Battery_Management:MCP73831-2-OT
- removed U?: LM7806_TO220, Package_TO_SOT_THT:TO-220-3_Vertical, symbol Regulator_Linear:LM7806_TO220
- added C1, C17, C2, C6: 4.7uF, symbol Device:C_Small
- added C10, C13, C15, C7: 10uF, symbol Device:C_Small
- added C11, C9: 0.01uF, symbol Device:C_Small
- added C12, C18, C8: 2.2uF, symbol Device:C_Small
- added C14, C4, C5: 0.1uF, symbol Device:C_Small
- added C16, C19: 100uF, symbol Device:C_Small
- added C3: C_Small, symbol Device:C_Small
- added D1: LED, symbol Device:LED
- added J1: USB_C_Receptacle_PowerOnly_6P, symbol Connector:USB_C_Receptacle_PowerOnly_6P
- added L1, L?: 2.2uH, symbol Device:L
- added L2: 6.8uH, symbol Device:L_Small
- added Q1, Q2: NMOS, symbol Simulation_SPICE:NMOS
- added R1: 2k, symbol Device:R_Small
- added R10, R6: 120k, symbol Device:R_Small
- added R11: R_Small, symbol Device:R_Small
- added R2: 470, symbol Device:R_Small
- added R3: 1k, symbol Device:R_Small
- added R4, R?: 100, symbol Device:R_Small
- added R5, R9: 1.5M, symbol Device:R_Small
- added R7, R8: 0.4, symbol Device:R_Small
- added R?: 0.1, symbol Device:R_Small
- added U1: MCP73831-2-OT, Package_TO_SOT_SMD:SOT-23-5, symbol Battery_Management:MCP73831-2-OT
- added U2: LM78M05_TO220, Package_TO_SOT_THT:TO-220-3_Vertical, symbol Regulator_Linear:LM78M05_TO220
- added U3: TPS61202DRC, Package_SON:Texas_S-PVSON-N10_ThermalVias, symbol Regulator_Switching:TPS61202DRC
- added U4: DW01A, Package_TO_SOT_SMD:SOT-23-6, symbol Battery_Management:DW01A
- added U5, U6: DRV8833PW, Package_SO:TSSOP-16_4.4x5mm_P0.65mm, symbol Driver_Motor:DRV8833PW
- added U7: TPS61092, Package_DFN_QFN:Texas_RSA_VQFN-16-1EP_4x4mm_P0.65mm_EP2.7x2.7mm_ThermalVias, symbol Regulator_Switching:TPS61092
- added U?: TPS63001, Package_SON:Texas_DRC0010J_ThermalVias, symbol Regulator_Switching:TPS63001
Connections:
- net 3v3in is gone; now on net 3V3: U?.8 (IN+)
- net Earth: now also C16.2, J1.A12 (GND), J1.B12 (GND), J1.S1 (SHIELD)
- net GND: now also U?.6 (GND), C1.2, C12.1, C17.2, C2.2, C5.2, C6.2, C8.1, R1.2, R10.2, R6.2, R7.1, R8.1, U1.2 (VSS), U2.2 (GND), U5.13 (GND), U6.13 (GND), U7.10 (SYNC), U7.13 (GND), U7.17 (PAD), U7.5 (PGND), U7.6 (PGND), U7.7 (PGND)
- net Vout_3.3v: now also C15.1, C16.1, U?.1 (VOUT), U?.10 (FB)
- net at U?.2 (A0): no longer U?.6 (GND)
- net 3V3: now reaches U?.5 (VS)
- net 3V3: now also C17.1, C6.1, C7.1, L1.1, L2.1, R4.1, R5.1, R9.1, R?.1, R?.1, U3.5 (VIN), U3.6 (EN), U3.8 (PS), U7.11 (EN), U7.8 (VBAT), U?.5 (VIN)
- net 3v3 out: no longer names the net of U?.1 (A1)
- net INA219 out renamed B-
- net B-: now also C4.2, Q1.1 (D), Q1.3 (S), Q2.1 (D), Q2.3 (S), R3.2, R?.2, U4.6 (GND)
- net pin3: no longer names the net of U?.4 (SCL)
- net pin4: no longer names the net of U?.3 (SDA)
- new net: C12.2, U6.14 (VINT)
- new net: R5.2, R6.1, U3.7 (UVLO)
- new net: C14.1, R?.2, U?.6 (EN), U?.7 (PS/SYNC), U?.8 (VINA)
- new net: R10.1, R9.2, U7.9 (LBI)
- new net: C2.1, D1.2 (A), U1.4 (VDD), U2.3 (VO)
- new net: C10.1, C9.1, U5.12 (VM)
- new net: C9.2, U5.11 (VCP)
- new net: D1.1 (K), R2.1
- new net: R3.1, U4.2 (CS)
- new net: R7.2, U5.3 (AISEN), U5.6 (BISEN)
- new net: C8.2, U5.14 (VINT)
- new net: Q2.2 (G), U4.3 (OC)
- new net: L2.2, U7.3 (SW), U7.4 (SW)
- new net: R8.2, U6.3 (AISEN), U6.6 (BISEN)
- new net: C11.1, C13.1, U6.12 (VM)
- new net: C11.2, U6.11 (VCP)
- new net: J1.A5 (CC1), J1.B5 (CC2)
- new net: R11.2, U7.12 (LBO)
- new net: C5.1, U3.1 (VAUX)
- new net: U3.11 (PAD), U3.4 (PGND), U3.9 (GND)
- new net: L1.2, U3.3 (L)
- new net: Q1.2 (G), U4.1 (OD)
- new net: C4.1, R4.2, U4.5 (VCC)
- new net: R1.1, U1.5 (PROG)
- new net: U?.11 (PGND), U?.3 (PGND), U?.9 (GND)
- new net: L?.2, U?.2 (L2)
- new net: L?.1, U?.4 (L1)
- new net: R2.2, U1.1 (STAT)
- new net 5V 2A: C18.1, C19.1, R11.1, U7.1 (VOUT), U7.14 (FB), U7.15 (VOUT), U7.16 (VOUT)
- new net 5V_out: U3.10 (FB), U3.2 (VOUT)
- new net 9V: J1.A9 (VBUS), J1.B9 (VBUS)
- new net AIN1: U5.16 (AIN1)
- new net AIN2: U5.15 (AIN2)
- new net AOUT1: U5.2 (AOUT1)
- new net AOUT2: U5.4 (AOUT2)
- new net B+ 500mA: C1.1, U1.3 (VBAT)
- new net BIN1: U5.9 (BIN1)
- new net BIN2: U5.10 (BIN2)
- new net BOUT1: U5.7 (BOUT1)
- new net BOUT2: U5.5 (BOUT2)
- new net CIN1: U6.16 (AIN1)
- new net CIN2: U6.15 (AIN2)
- new net COUT1: U6.2 (AOUT1)
- new net COUT2: U6.4 (AOUT2)
- new net DIN1: U6.9 (BIN1)
- new net DIN2: U6.10 (BIN2)
- new net DOUT1: U6.7 (BOUT1)
- new net DOUT2: U6.5 (BOUT2)
- new net SLEEP: U5.1 (nSLEEP), U6.1 (nSLEEP)
- new net Vin_9V: C3.1, U2.1 (VI)
- no-connect marks 5 -> 0
Other:
- note removed: "200mA output"
- note removed: "500mA out"
- note removed: "Charging circuit"
- note removed: "motor controll"
- note removed: "when battery output is 3.2, vout drops to zero"
- moved on the sheet: J?, U?

Commit message: Add files via upload
Parts:
- added C20: 1uF, symbol Device:C_Small
- added C21: 10uF, symbol Device:C_Small
- added Q3: NMOS, symbol Simulation_SPICE:NMOS
- added R12, R13: 5.1k, symbol Device:R_Small
- added R14: 4.7k, symbol Device:R_Small
- added SW1, SW2, SW3: SW_Push, symbol Switch:SW_Push
- added U8: IP2721, Package_SO:TSSOP-16_4.4x5mm_P0.65mm, symbol Interface_USB:IP2721
Connections:
- net 3V3: now also SW1.1; no longer C17.1, C7.1, L2.1, R9.1, R?.1, U7.11 (EN), U7.8 (VBAT), U?.5 (VIN)
- net 9V: now also C20.1, C21.1, Q3.1 (D), Q3.3 (S), U8.16 (VBUS)
- net GND: now also R14.1
- net at J1.B5 (CC2): now also R12.1, U8.12 (CC2); no longer J1.A5 (CC1)
- net at U1.5 (PROG): now also SW2.1, SW3.1; no longer R1.1
- net B+ 500mA renamed B+ 
- new net: R14.2, SW3.2
- new net: Q3.2 (G), U8.1 (VBUSG)
- new net: J1.A5 (CC1), R13.2, U8.13 (CC1)
- new net: R1.1, SW2.2
- new net Vin: C17.1, C7.1, L2.1, R9.1, R?.1, SW1.2, U7.11 (EN), U7.8 (VBAT), U?.5 (VIN)
Other:
- moved on the sheet: C1, C2, C3, D1, J1, R1, R2, U1, U2

Commit message: Add files via upload
Connections:
- net AIN1 is gone; now on net motor2_CTRL1: U5.16 (AIN1)
- net AIN2 is gone; now on net motor2_CTRL2: U5.15 (AIN2)
- net AOUT1 is gone; now on net motor2_A_out: U5.2 (AOUT1)
- net AOUT2 is gone; now on net motor2_B_out: U5.4 (AOUT2)
- net BIN1 is gone; now on net motor4_CTRL1: U5.9 (BIN1)
- net BIN2 is gone; now on net motor4_CTRL2: U5.10 (BIN2)
- net BOUT1 is gone; now on net motor4_A_out: U5.7 (BOUT1)
- net BOUT2 is gone; now on net motor4_B_out: U5.5 (BOUT2)
- net CIN1 is gone; now on net motor1_CTRL1: U6.16 (AIN1)
- net CIN2 is gone; now on net motor1_CTRL2: U6.15 (AIN2)
- net DIN1 is gone; now on net motor3_CTRL1: U6.9 (BIN1)
- net DIN2 is gone; now on net motor3_CTRL2: U6.10 (BIN2)
- net COUT1 renamed motor1_A_out
- net COUT2 renamed motor1_B_out
- net DOUT1 renamed motor3_A_out
- net DOUT2 renamed motor3_B_out
Other:
- moved on the sheet: J?
Changed lines of the file:
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@@
 	(text_box "Motor powering\n"
 		(exclude_from_sim no)
-		(at 152.4 12.7 0)
+		(at 149.86 12.7 0)
 		(size 132.08 68.58)
 		(margins 0.9525 0.9525 0.9525 0.9525)
@@
 		)
 	)
-	(label "BOUT1"
+	(label "motor4_A_out"
 		(at 262.89 58.42 0)
 		(effects
@@
 		)
 	)
-	(label "BOUT2"
+	(label "motor4_B_out"
 		(at 262.89 60.96 0)
 		(effects
@@
 	)
 	(label "motor4_CTRL1"
-		(at 45.72 194.31 270)
+		(at 44.45 162.56 180)
 		(effects
 			(font
@@
 		)
 	)
-	(label "AOUT2"
+	(label "motor2_B_out"
 		(at 262.89 55.88 0)
 		(effects
@@
 	)
 	(label "GND"
-		(at 60.96 181.61 90)
+		(at 57.15 177.8 0)
 		(effects
 			(font
@@
 	)
 	(label "motor4_B_out"
-		(at 43.18 181.61 90)
+		(at 57.15 160.02 0)
 		(effects
 			(font
@@
 		)
 	)
-	(label "AIN1"
+	(label "motor2_CTRL1"
 		(at 227.33 53.34 0)
 		(effects
@@
 		)
 	)
-	(label "AOUT1"
+	(label "motor2_A_out"
 		(at 262.89 53.34 0)
 		(effects
@@
 		)
 	)
-	(label "CIN1"
+	(label "motor1_CTRL1"
 		(at 171.45 55.88 0)
 		(effects
@@
 	)
 	(label "motor1_A_OUT"
-		(at 76.2 194.31 270)
+		(at 44.45 193.04 180)
 		(effects
 			(font
@@
 	)
 	(label "EXT_LOAD2_OUT"
-		(at 50.8 181.61 90)
+		(at 57.15 167.64 0)
 		(effects
 			(font
@@
 		)
 	)
-	(label "BIN1"
+	(label "motor4_CTRL1"
 		(at 227.33 58.42 0)
 		(effects
@@
 		)
 	)
-	(label "CIN2"
+	(label "motor1_CTRL2"
 		(at 171.45 58.42 0)
 		(effects
@@
 	)
 	(label "motor2_CTRL1"
-		(at 40.64 194.31 270)
+		(at 44.45 157.48 180)
 		(effects
 			(font
@@
 		)
 	)
-	(label "DIN1"
+	(label "motor3_CTRL1"
 		(at 171.45 60.96 0)
 		(effects
@@
 		)
 	)
-	(label "DOUT1"
+	(label "motor3_A_out"
 		(at 207.01 60.96 0)
 		(effects
@@
 	)
 	(label "GND"
-		(at 66.04 181.61 90)
+		(at 57.15 182.88 0)
 		(effects
 			(font
@@
 	)
 	(label "USART2_RX"
-		(at 48.26 181.61 90)
+		(at 57.15 165.1 0)
 		(effects
 			(font
@@
 	)
 	(label "motor3_CTRL2"
-		(at 68.58 194.31 270)
+		(at 44.45 185.42 180)
 		(effects
 			(font
@@
 	)
 	(label "USART2_TX"
-		(at 50.8 194.31 270)
+		(at 44.45 167.64 180)
 		(effects
 			(font
@@
 	)
 	(label "motor2_CTRL2"
-		(at 43.18 194.31 270)
+		(at 44.45 160.02 180)
 		(effects
 			(font
@@
 	)
 	(label "I2C1_SDA"
-		(at 58.42 181.61 90)
+		(at 57.15 175.26 0)
 		(effects
 			(font
@@
 		)
 	)
-	(label "DOUT2"
+	(label "motor3_B_out"
 		(at 207.01 63.5 0)
 		(effects
@@
 	)
 	(label "motor2_A_out"
-		(at 38.1 194.31 270)
+		(at 44.45 154.94 180)
 		(effects
 			(font
@@
 		)
 	)
-	(label "COUT1"
+	(label "motor1_A_out"
 		(at 207.01 55.88 0)
 		(effects
@@
 	)
 	(label "HV"
-		(at 63.5 194.31 270)
+		(at 44.45 180.34 180)
 		(effects
 			(font
@@
 	)
 	(label "motor1_B_OUT"
-		(at 76.2 181.61 90)
+		(at 57.15 193.04 0)
 		(effects
 			(font
@@
 	)
 	(label "."
-		(at 55.88 181.61 90)
+		(at 57.15 172.72 0)
 		(effects
 			(font
@@
 	)
 	(label "motor3_CTRL1"
-		(at 66.04 194.31 270)
+		(at 44.45 182.88 180)
 		(effects
 			(font
@@
 	)
 	(label "FAST_CHARGE_CTRL"
-		(at 53.34 181.61 90)
+		(at 57.15 170.18 0)
 		(effects
 			(font
@@
 	)
 	(label "CTRL_EXT_LOAD2"
-		(at 45.72 181.61 90)
+		(at 57.15 162.56 0)
 		(effects
 			(font
@@
 	)
 	(label "motor4_CTRL2"
-		(at 48.26 194.31 270)
+		(at 44.45 165.1 180)
 		(effects
 			(font
@@
 	)
 	(label "motor1_CTRL2"
-		(at 73.66 194.31 270)
+		(at 44.45 190.5 180)
 		(effects
 			(font
@@
 	)
 	(label "I2C1_SCL"
-		(at 55.88 194.31 270)
+		(at 44.45 172.72 180)
 		(effects
 			(font
@@
 		)
 	)
-	(label "DIN2"
+	(label "motor3_CTRL2"
 		(at 171.45 63.5 0)
 		(effects
@@
 	)
 	(label "motor1_CTRL1"
-		(at 71.12 194.31 270)
+		(at 44.45 187.96 180)
 		(effects
 			(font
@@
 	)
 	(label "CTRL_EXT_LOAD1"
-		(at 68.58 181.61 90)
+		(at 57.15 185.42 0)
 		(effects
 			(font
@@
 	)
 	(label "motor3_B_OUT"
-		(at 73.66 181.61 90)
+		(at 57.15 190.5 0)
 		(effects
 			(font
@@
 	)
 	(label "motor2_B_out"
-		(at 38.1 181.61 90)
+		(at 57.15 154.94 0)
 		(effects
 			(font
@@
 		)
 	)
-	(label "AIN2"
+	(label "motor2_CTRL2"
 		(at 227.33 55.88 0)
 		(effects
@@
 	)
 	(label "motor4_A_out"
-		(at 40.64 181.61 90)
+		(at 57.15 157.48 0)
 		(effects
 			(font
@@
 	)
 	(label "EXT_LOAD1_OUT"
-		(at 63.5 181.61 90)
+		(at 57.15 180.34 0)
 		(effects
 			(font
@@
 	)
 	(label "5V out"
-		(at 60.96 194.31 270)
+		(at 44.45 177.8 180)
 		(effects
 			(font
@@
 	)
 	(label "Battery"
-		(at 53.34 194.31 270)
+		(at 44.45 170.18 180)
 		(effects
 			(font
@@
 		)
 	)
-	(label "COUT2"
+	(label "motor1_B_out"
 		(at 207.01 58.42 0)
 		(effects
@@
 	)
 	(label "3V3 out"
-		(at 58.42 194.31 270)
+		(at 44.45 175.26 180)
 		(effects
 			(font
@@
 		)
 	)
-	(label "BIN2"
+	(label "motor4_CTRL2"
 		(at 227.33 60.96 0)
 		(effects
@@
 	)
 	(label "motor3_A_OUT"
-		(at 71.12 181.61 90)
+		(at 57.15 187.96 0)
 		(effects
 			(font
@@
 	(symbol
 		(lib_id "Connector_Generic:Conn_02x16_Odd_Even")
-		(at 55.88 186.69 90)
-		(mirror x)
+		(at 52.07 172.72 0)
+		(mirror y)
 		(unit 1)
 		(exclude_from_sim no)
@@
 		(fields_autoplaced yes)
 		(property "Reference" "J?"
-			(at 78.74 189.2301 90)
+			(at 52.0701 152.4 90)
 			(effects
 				(font
 					(size 1.27 1.27)
 				)
-				(justify right)
+				(justify left)
 			)
 		)
 		(property "Value" "Conn_02x16_Odd_Even"
-			(at 78.74 186.6901 90)
+			(at 49.5301 152.4 90)
 			(effects
 				(font
 					(size 1.27 1.27)
 				)
-				(justify right)
+				(justify left)
 			)
 		)
 		(property "Footprint" ""
-			(at 55.88 186.69 0)
+			(at 52.07 172.72 0)
 			(effects
 				(font
@@
 		)
 		(property "Datasheet" "~"
-			(at 55.88 186.69 0)
+			(at 52.07 172.72 0)
 			(effects
 				(font
@@
 		)
 		(property "Description" ""
-			(at 55.88 186.69 0)
+			(at 52.07 172.72 0)
 			(effects
 				(font

Commit message: Add files via upload
Parts:
- removed C5: 0.1uF, symbol Device:C_Small
- removed C6: 4.7uF, symbol Device:C_Small
- removed L1: 2.2uH, symbol Device:L
- removed R5: 1.5M, symbol Device:R_Small
- removed R6: 120k, symbol Device:R_Small
- removed U3: TPS61202DRC, Package_SON:Texas_S-PVSON-N10_ThermalVias, symbol Regulator_Switching:TPS61202DRC
- added BT1: Battery, symbol Device:Battery
- added TP1, TP10, TP11, TP12, TP13, TP14, TP15, TP16, TP2, TP3, TP4, TP5, TP6, TP7, TP8, TP9: TestPoint, TestPoint:TestPoint_Pad_1.5x1.5mm, symbol Connector:TestPoint
- C1, C10, C11, C12, C13, C14, C15, C16, C17, C18, C19, C2, C20, C21, C4, C7, C8, C9: footprint (none) -> Capacitor_THT:C_Disc_D3.0mm_W1.6mm_P2.50mm
- C3: value C_Small -> 1uF; footprint (none) -> Capacitor_THT:C_Disc_D3.0mm_W1.6mm_P2.50mm
- D1: footprint (none) -> LED_THT:LED_D2.0mm_W4.0mm_H2.8mm_FlatTop
- J2: renamed from J?; footprint (none) -> Connector_PinHeader_1.00mm:PinHeader_2x16_P1.00mm_Horizontal
- L2: footprint (none) -> Inductor_THT:L_Axial_L5.0mm_D3.6mm_P10.00mm_Horizontal_Murata_BL01RN1A2A2
- L3: renamed from L?; footprint (none) -> Inductor_THT:L_Axial_L5.0mm_D3.6mm_P10.00mm_Horizontal_Murata_BL01RN1A2A2
- R1, R10, R12, R13, R14, R2, R3, R4, R9: footprint (none) -> Resistor_THT:R_Axial_DIN0204_L3.6mm_D1.6mm_P1.90mm_Vertical
- R11: value R_Small -> 100k; footprint (none) -> Resistor_THT:R_Axial_DIN0204_L3.6mm_D1.6mm_P1.90mm_Vertical
- R15, R16: renamed from R?; footprint (none) -> Resistor_THT:R_Axial_DIN0204_L3.6mm_D1.6mm_P1.90mm_Vertical
- R7, R8: value 0.4 -> 0.7; footprint (none) -> Resistor_THT:R_Axial_DIN0204_L3.6mm_D1.6mm_P1.90mm_Vertical
- SW1, SW2, SW3: footprint (none) -> Button_Switch_THT:SW_PUSH_6mm_H4.3mm
- gave numbers to parts that had none: 2
Connections:
- net 5V 2A is gone; now on net 5V out: C18.1, C19.1, R11.1, U7.1 (VOUT), U7.14 (FB), U7.15 (VOUT), U7.16 (VOUT)
- net B- is gone; now on net Earth: C4.2, Q1.1 (D), Q1.3 (S), Q2.1 (D), Q2.3 (S), R15.2, R3.2, U4.6 (GND), U9.7 (IN-)
- net GND is gone; now on net Earth: C1.2, C12.1, C17.2, C2.2, C8.1, J2.19 (Pin_19), J2.23 (Pin_23), R1.2, R10.2, R14.1, R7.1, R8.1, U1.2 (VSS), U2.2 (GND), U5.13 (GND), U6.13 (GND), U7.10 (SYNC), U7.13 (GND), U7.17 (PAD), U7.5 (PGND), U7.6 (PGND), U7.7 (PGND), U9.6 (GND)
- net 3V3: now also BT1.1 (+)
- net 5V out: now also TP5.1
- net B+ : now also TP6.1
- net Earth: now also C14.2, C15.2, C18.2, C19.2, C20.2, C21.2, C7.2, R11.2, R12.2, R13.1, U10.11 (PGND), U10.3 (PGND), U10.9 (GND), U7.12 (LBO), U8.5 (GND), BT1.2 (-), TP14.1, TP16.1
- net Vin_9V: now also TP7.1
- net at C14.1, R16.2, U10.6 (EN)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: now also TP3.1
- net at C2.1, D1.2 (A), U1.4 (VDD)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: now also TP11.1
- net at R7.2, U5.3 (AISEN), U5.6 (BISEN): now also TP15.1
- net at R8.2, U6.3 (AISEN), U6.6 (BISEN): now also TP13.1
- net 9V renamed Vout_9V
- net Vout_9V: now also TP12.1, TP4.1
- net Vin renamed Vin_3.7V
- net Vin_3.7V: now also TP2.1, TP8.1, TP9.1
- net Vout_3.3v renamed 3V3 oit
- net 3V3 oit: now also TP10.1
Other:
- moved on the sheet: C1, SW1
